File: Tarea_2_unai/Microcontrolador.kicad_sch (KiCad schematic)
At the start: 5 parts, among them IC1 ESP32-C3-MINI-1-N4

Commit message: actuacilación
Parts:
- added J2: Conn_01x02_Pin, PinHeader_1x04_P2.54mm_Vertical, symbol Connector:Conn_01x02_Pin
- IC1: footprint ESP32C3MINI1N4 -> ESP32-C3-MINI-1-N4
Connections:
- net GND_REF: now also J2.1 (Pin_1); no longer IC1.5 (IO2)
- net at C1.1, R1.1: now also J2.2 (Pin_2); no longer IC1.7 (NC_2)
- no-connect marks 56 -> 58
Changed lines of the file:
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@@
+	)
+	(junction
+		(at 68.58 72.39)
+		(diameter 0)
+		(color 0 0 0 0)
 	)
 	(junction
@@
 		(color 0 0 0 0)
 	)
-	(junction
-		(at 68.58 81.28)
-		(diameter 0)
-		(color 0 0 0 0)
-	)
 	(no_connect
 		(at 119.38 74.93)
@@
 	)
 	(no_connect
+		(at 119.38 36.83)
+	)
+	(no_connect
 		(at 152.4 95.25)
 	)
@@
 	)
 	(no_connect
+		(at 119.38 31.75)
+	)
+	(no_connect
 		(at 152.4 72.39)
 	)
@@
 	(wire
 		(pts
+			(xy 71.12 58.42) (xy 71.12 67.31)
+		)
+		(stroke
+			(width 0)
+			(type default)
+		)
+	)
+	(wire
+		(pts
 			(xy 118.11 26.67) (xy 119.38 26.67)
 		)
@@
 	(wire
 		(pts
-			(xy 119.38 36.83) (xy 100.33 36.83)
-		)
-		(stroke
-			(width 0)
-			(type default)
-		)
-	)
-	(wire
-		(pts
 			(xy 118.11 25.4) (xy 85.09 25.4)
 		)
@@
 	(wire
 		(pts
-			(xy 100.33 36.83) (xy 100.33 81.28)
-		)
-		(stroke
-			(width 0)
-			(type default)
-		)
-	)
-	(wire
-		(pts
 			(xy 85.09 58.42) (xy 85.09 29.21)
 		)
@@
 	(wire
 		(pts
-			(xy 68.58 72.39) (xy 68.58 81.28)
-		)
-		(stroke
-			(width 0)
-			(type default)
-		)
-	)
-	(wire
-		(pts
-			(xy 119.38 31.75) (xy 88.9 31.75)
+			(xy 68.58 69.85) (xy 68.58 72.39)
+		)
+		(stroke
+			(width 0)
+			(type default)
+		)
+	)
+	(wire
+		(pts
+			(xy 68.58 72.39) (xy 68.58 82.55)
 		)
 		(stroke
@@
 	(wire
 		(pts
-			(xy 71.12 58.42) (xy 71.12 66.04)
-		)
-		(stroke
-			(width 0)
-			(type default)
-		)
-	)
-	(wire
-		(pts
-			(xy 100.33 81.28) (xy 68.58 81.28)
-		)
-		(stroke
-			(width 0)
-			(type default)
-		)
-	)
-	(wire
-		(pts
 			(xy 30.48 97.79) (xy 68.58 97.79)
 		)
@@
 	(wire
 		(pts
-			(xy 88.9 31.75) (xy 88.9 66.04)
-		)
-		(stroke
-			(width 0)
-			(type default)
-		)
-	)
-	(wire
-		(pts
-			(xy 68.58 81.28) (xy 68.58 82.55)
-		)
-		(stroke
-			(width 0)
-			(type default)
-		)
-	)
-	(wire
-		(pts
-			(xy 88.9 66.04) (xy 71.12 66.04)
+			(xy 64.77 69.85) (xy 68.58 69.85)
+		)
+		(stroke
+			(width 0)
+			(type default)
+		)
+	)
+	(wire
+		(pts
+			(xy 71.12 67.31) (xy 64.77 67.31)
 		)
 		(stroke
@@
 			)
 		)
-		(property "Footprint" "ESP32C3MINI1N4"
+		(property "Footprint" "ESP32-C3-MINI-1-N4"
 			(at 148.59 116.51 0)
 			(hide yes)
@@
 					(unit 1)
 				)
+			)
+		)
+	)
+	(symbol
+		(lib_id "Connector:Conn_01x02_Pin")
+		(at 59.69 67.31 0)
+		(unit 1)
+		(body_style 1)
+		(exclude_from_sim no)
+		(in_bom yes)
+		(on_board yes)
+		(in_pos_files yes)
+		(dnp no)
+		(fields_autoplaced yes)
+		(property "Reference" "J2"
+			(at 60.325 62.23 0)
+			(show_name no)
+			(do_not_autoplace no)
+			(effects
+				(font
+					(size 1.27 1.27)
+				)
+			)
+		)
+		(property "Value" "Conn_01x02_Pin"
+			(at 60.325 64.77 0)
+			(show_name no)
+			(do_not_autoplace no)
+			(effects
+				(font
+					(size 1.27 1.27)
+				)
+			)
+		)
+		(property "Footprint" "PinHeader_1x04_P2.54mm_Vertical"
+			(at 59.69 67.31 0)
+			(hide yes)
+			(show_name no)
+			(do_not_autoplace no)
+			(effects
+				(font
+					(size 1.27 1.27)
+				)
+			)
+		)
+		(property "Datasheet" ""
+			(at 59.69 67.31 0)
+			(hide yes)
+			(show_name no)
+			(do_not_autoplace no)
+			(effects
+				(font
+					(size 1.27 1.27)
+				)
+			)
+		)
+		(property "Description" "Generic connector, single row, 01x02, script generated"
+			(at 59.69 67.31 0)
+			(hide yes)
+			(show_name no)
+			(do_not_autoplace no)
+			(effects
+				(font
+					(size 1.27 1.27)
+				)
+			)
+		)
+		(pin "2"
+		)
+		(pin "1"
+		)
+		(instances
+			(project "Tarea_2_unai"
+				(path "/2324ac65-aae7-4e51-a8e4-9d93764ceb90/5cbed766-6105-4833-8b7f-4c3640c40f4a"
+					(reference "J2")
+					(unit 1)
+				)
