File: Tarea_2_unai/Tarea_2_unai.kicad_sch (KiCad schematic)
At the start: 0 parts

Commit message: actualización completa
Changed lines of the file:
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@@
 			)
 		)
-		(pin "GND_REF" output
+		(pin "GND_REF" input
 			(at 83.82 63.5 0)
 			(effects
@@
 			)
 		)
-		(pin "VOUT_3V3" output
+		(pin "VOUT_3V3" input
 			(at 83.82 53.34 0)
 			(effects
