File: Tarea_2_unai/Tarea_2_unai.kicad_pcb (KiCad board)
At the start: 2 copper layers, 44.5 x 31.5 mm, 10 parts, among them IC2 ESP32-C3-MINI-1-N4X, J1 Conn_01x02_Pin, J2 Conn_01x02_Pin, U1 AMS1117-3.3

Commit message: enrutado
Routing:
- net /Alimentacion/GND_REF: track 0.00 -> 54.4 mm
- net /Alimentacion/VOUT_3V3: track 0.00 -> 17.1 mm, vias 0 -> 2
- net Net-(J1-Pin_1): track 0.00 -> 7.17 mm
- net Net-(IC2-NC_1): track 0.00 -> 5.89 mm
- net Net-(J2-Pin_2): track 0.00 -> 5.78 mm
- net Net-(J2-Pin_1): track 0.00 -> 4.74 mm
- net Net-(IC2-IO3): track 0.00 -> 3.79 mm

Commit message: zona_fill
Parts:
- moved R2 0.20 mm to (129.5, 96.5), turned to 180 degrees
Connections:
- IC2 pad 11: unconnected-(IC2-GND_3-Pad11) -> /Alimentacion/GND_REF
- IC2 pad 14: unconnected-(IC2-GND_4-Pad14) -> /Alimentacion/GND_REF
- IC2 pad 2: unconnected-(IC2-GND_2-Pad2) -> /Alimentacion/GND_REF
Routing:
- net /Alimentacion/GND_REF: track 54.4 -> 0.29 mm
- net /Alimentacion/VOUT_3V3: track 17.1 -> 18.0 mm, vias 2 -> 0
- net Net-(J2-Pin_2): track 5.78 -> 4.93 mm
- added copper zone on F.Cu, net /Alimentacion/GND_REF
